File: kicad/Valmer 1.kicad_pcb (KiCad board)
At the start: 4 copper layers, 74 parts

Commit message: kicad update
Parts:
- added LED1: Placeholder_LED, LED_SMD:LED_0603_1608Metric, F.Cu at (219.5, 77.1)
- added LED10: Placeholder_LED, LED_SMD:LED_0603_1608Metric, F.Cu at (230.2, 83.1)
- added LED11: Placeholder_LED, LED_SMD:LED_0603_1608Metric, F.Cu at (230.2, 85.7)
- added LED12: Placeholder_LED, LED_SMD:LED_0603_1608Metric, F.Cu at (230.2, 88.3)
- added LED13: Placeholder_LED, LED_SMD:LED_0603_1608Metric, F.Cu at (230.2, 90.9)
- added LED14: Placeholder_LED, LED_SMD:LED_0603_1608Metric, F.Cu at (230.2, 93.5)
- added LED15: Placeholder_LED, LED_SMD:LED_0603_1608Metric, F.Cu at (230.2, 96.1)
- added LED16: Placeholder_LED, LED_SMD:LED_0603_1608Metric, F.Cu at (230.2, 98.7)
- added LED17: Placeholder_LED, LED_SMD:LED_0603_1608Metric, F.Cu at (234.3, 80.5)
- added LED18: Placeholder_LED, LED_SMD:LED_0603_1608Metric, F.Cu at (234.3, 83.1)
- added LED19: Placeholder_LED, LED_SMD:LED_0603_1608Metric, F.Cu at (234.3, 85.7)
- added LED2: Placeholder_LED, LED_SMD:LED_0603_1608Metric, F.Cu at (226.2, 83.1)
- added LED20: Placeholder_LED, LED_SMD:LED_0603_1608Metric, F.Cu at (234.3, 88.3)
- added LED21: Placeholder_LED, LED_SMD:LED_0603_1608Metric, F.Cu at (234.3, 90.9)
- added LED22: Placeholder_LED, LED_SMD:LED_0603_1608Metric, F.Cu at (234.3, 93.5)
- added LED23: Placeholder_LED, LED_SMD:LED_0603_1608Metric, F.Cu at (234.3, 96.1)
- added LED24: Placeholder_LED, LED_SMD:LED_0603_1608Metric, F.Cu at (234.3, 98.7)
- added LED25: Placeholder_LED, LED_SMD:LED_0603_1608Metric, F.Cu at (238.3, 80.5)
- added LED26: Placeholder_LED, LED_SMD:LED_0603_1608Metric, F.Cu at (238.3, 83.1)
- added LED27: Placeholder_LED, LED_SMD:LED_0603_1608Metric, F.Cu at (238.3, 85.7)
- added LED28: Placeholder_LED, LED_SMD:LED_0603_1608Metric, F.Cu at (238.3, 88.3)
- added LED29: Placeholder_LED, LED_SMD:LED_0603_1608Metric, F.Cu at (238.3, 90.9)
- added LED3: Placeholder_LED, LED_SMD:LED_0603_1608Metric, F.Cu at (226.2, 85.7)
- added LED30: Placeholder_LED, LED_SMD:LED_0603_1608Metric, F.Cu at (238.3, 93.5)
- added LED31: Placeholder_LED, LED_SMD:LED_0603_1608Metric, F.Cu at (238.3, 96.1)
- added LED32: Placeholder_LED, LED_SMD:LED_0603_1608Metric, F.Cu at (238.3, 98.7)
- added LED33: Placeholder_LED, LED_SMD:LED_0603_1608Metric, F.Cu at (242.4, 80.5)
- added LED34: Placeholder_LED, LED_SMD:LED_0603_1608Metric, F.Cu at (242.4, 83.1)
- added LED35: Placeholder_LED, LED_SMD:LED_0603_1608Metric, F.Cu at (242.4, 85.7)
- added LED36: Placeholder_LED, LED_SMD:LED_0603_1608Metric, F.Cu at (242.4, 88.3)
- added LED37: Placeholder_LED, LED_SMD:LED_0603_1608Metric, F.Cu at (242.4, 90.9)
- added LED4: Placeholder_LED, LED_SMD:LED_0603_1608Metric, F.Cu at (226.2, 88.3)
- added LED5: Placeholder_LED, LED_SMD:LED_0603_1608Metric, F.Cu at (226.2, 90.9)
- added LED6: Placeholder_LED, LED_SMD:LED_0603_1608Metric, F.Cu at (226.2, 93.5)
- added LED7: Placeholder_LED, LED_SMD:LED_0603_1608Metric, F.Cu at (226.2, 96.1)
- added LED8: Placeholder_LED, LED_SMD:LED_0603_1608Metric, F.Cu at (226.2, 98.7)
- added LED9: Placeholder_LED, LED_SMD:LED_0603_1608Metric, F.Cu at (230.2, 80.5)
- added R1: 1K, Resistor_SMD:R_0603_1608Metric, F.Cu at (246.4, 80.5)
- added R10: 1K, Resistor_SMD:R_0603_1608Metric, F.Cu at (250.4, 83.0)
- added R11: 1K, Resistor_SMD:R_0603_1608Metric, F.Cu at (250.4, 85.5)
- added R12: 1K, Resistor_SMD:R_0603_1608Metric, F.Cu at (250.4, 88.0)
- added R13: 1K, Resistor_SMD:R_0603_1608Metric, F.Cu at (250.4, 90.5)
- added R14: 1K, Resistor_SMD:R_0603_1608Metric, F.Cu at (250.4, 93.0)
- added R15: 1K, Resistor_SMD:R_0603_1608Metric, F.Cu at (250.4, 95.6)
- added R16: 1K, Resistor_SMD:R_0603_1608Metric, F.Cu at (250.4, 98.1)
- added R17: 1K, Resistor_SMD:R_0603_1608Metric, F.Cu at (254.4, 80.5)
- added R18: 1K, Resistor_SMD:R_0603_1608Metric, F.Cu at (254.4, 83.0)
- added R19: 1K, Resistor_SMD:R_0603_1608Metric, F.Cu at (254.4, 85.5)
- added R2: 1K, Resistor_SMD:R_0603_1608Metric, F.Cu at (246.4, 83.0)
- added R20: 1K, Resistor_SMD:R_0603_1608Metric, F.Cu at (254.4, 88.0)
- added R21: 1K, Resistor_SMD:R_0603_1608Metric, F.Cu at (254.4, 90.5)
- added R22: 1K, Resistor_SMD:R_0603_1608Metric, F.Cu at (254.4, 93.0)
- added R23: 1K, Resistor_SMD:R_0603_1608Metric, F.Cu at (254.4, 95.6)
- added R24: 1K, Resistor_SMD:R_0603_1608Metric, F.Cu at (254.4, 98.1)
- added R25: 1K, Resistor_SMD:R_0603_1608Metric, F.Cu at (258.4, 80.5)
- added R26: 1K, Resistor_SMD:R_0603_1608Metric, F.Cu at (258.4, 83.0)
- added R27: 1K, Resistor_SMD:R_0603_1608Metric, F.Cu at (258.4, 85.5)
- added R28: 1K, Resistor_SMD:R_0603_1608Metric, F.Cu at (258.4, 88.0)
- added R29: 1K, Resistor_SMD:R_0603_1608Metric, F.Cu at (258.4, 90.5)
- added R3: 1K, Resistor_SMD:R_0603_1608Metric, F.Cu at (246.4, 85.5)
- added R30: 1K, Resistor_SMD:R_0603_1608Metric, F.Cu at (258.4, 93.0)
- added R31: 1K, Resistor_SMD:R_0603_1608Metric, F.Cu at (258.4, 95.6)
- added R32: 1K, Resistor_SMD:R_0603_1608Metric, F.Cu at (258.4, 98.1)
- added R33: 1K, Resistor_SMD:R_0603_1608Metric, F.Cu at (262.4, 80.5)
- added R34: 1K, Resistor_SMD:R_0603_1608Metric, F.Cu at (262.4, 83.0)
- added R35: 1K, Resistor_SMD:R_0603_1608Metric, F.Cu at (262.4, 85.5)
- added R36: 1K, Resistor_SMD:R_0603_1608Metric, F.Cu at (262.4, 88.0)
- added R37: 1K, Resistor_SMD:R_0603_1608Metric, F.Cu at (262.4, 90.5)
- added R4: 1K, Resistor_SMD:R_0603_1608Metric, F.Cu at (246.4, 88.0)
- added R5: 1K, Resistor_SMD:R_0603_1608Metric, F.Cu at (246.4, 90.5)
- added R6: 1K, Resistor_SMD:R_0603_1608Metric, F.Cu at (246.4, 93.0)
- added R7: 1K, Resistor_SMD:R_0603_1608Metric, F.Cu at (246.4, 95.6)
- added R8: 1K, Resistor_SMD:R_0603_1608Metric, F.Cu at (246.4, 98.1)
- added R9: 1K, Resistor_SMD:R_0603_1608Metric, F.Cu at (250.4, 80.5)
- added U1: RP2040_Pro_Micro, ScottoKeebs_MCU:RP2040_Pro_Micro, F.Cu at (174.3, 81.1)
- D1, D10, D11, D12, D13, D14, D15, D16, D17, D18, D19, D2, D20, D21, D22, D23, D24, D25, D26, D27, D28, D29, D3, D30, D31, D32, D33, D34, D35, D36, D37, D4, D5, D6, D7, D8, D9: moved to B.Cu
- moved D30 158.1 mm to (42.8, 111.4), turned to 90 degrees
- moved D22 149.8 mm to (42.8, 94.4), turned to 90 degrees
- moved D15 143.3 mm to (42.8, 77.4), turned to 90 degrees
- moved D8 139.8 mm to (42.8, 60.4), turned to 90 degrees
- moved D1 138.8 mm to (42.8, 43.4), turned to 90 degrees
- moved D31 137.6 mm to (63.0, 111.4), turned to 90 degrees
- moved D23 129.3 mm to (63.0, 94.4), turned to 90 degrees
- moved D16 123.3 mm to (63.0, 77.4), turned to 90 degrees
- moved D9 123.0 mm to (63.0, 60.4), turned to 90 degrees
- moved D2 119.3 mm to (63.0, 43.4), turned to 90 degrees
- moved D32 118.4 mm to (81.0, 107.1), turned to 90 degrees
- moved S30 115.6 mm to (33.8, 108.4)
- moved S8 115.1 mm to (33.8, 57.4)
- moved D33 112.7 mm to (99.0, 105.0), turned to 90 degrees
- moved D17 111.3 mm to (81.0, 73.1), turned to 90 degrees
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Connections:
- D15 pad 1: Row 3 -> Row 2
- D16 pad 1: Row 3 -> Row 2
- D17 pad 1: Row 3 -> Row 2
- D18 pad 1: Row 3 -> Row 2
- D19 pad 1: Row 3 -> Row 2
- D20 pad 1: Row 3 -> Row 2
- D21 pad 1: Row 3 -> Row 2
- D22 pad 1: Row 4 -> Row 3
- D23 pad 1: Row 4 -> Row 3
- D24 pad 1: Row 4 -> Row 3
- D25 pad 1: Row 4 -> Row 3
- D26 pad 1: Row 4 -> Row 3
- D27 pad 1: Row 4 -> Row 3
- D28 pad 1: Row 4 -> Row 3
- D29 pad 1: Row 4 -> Row 3
- D30 pad 1: Row 5 -> Row 4
- D31 pad 1: Row 5 -> Row 4
- D32 pad 1: Row 5 -> Row 4
- D33 pad 1: Row 5 -> Row 4
- D34 pad 1: Row 5 -> Row 4
- D35 pad 1: Row 5 -> Row 4
- D36 pad 1: Row 5 -> Row 4
- D37 pad 1: Row 5 -> Row 4
Routing:
- net Colum 0: track 0.00 -> 252.9 mm
- net Colum 1: track 0.00 -> 234.9 mm
- net Row 3: track 0.00 -> 232.3 mm, vias 0 -> 8
- net Row 4: track 0.00 -> 232.1 mm, vias 0 -> 8
- net Colum 2: track 0.00 -> 217.5 mm
- net Colum 3: track 0.00 -> 202.2 mm
- net Colum 4: track 0.00 -> 184.4 mm
- net Colum 5: track 0.00 -> 183.8 mm
- net Colum 6: track 0.00 -> 172.9 mm
- net Row 0: track 0.00 -> 172.7 mm, vias 0 -> 7
- net Row 2: track 0.00 -> 159.8 mm, vias 0 -> 7
- net Row 1: track 0.00 -> 153.4 mm, vias 0 -> 7
- net Colum 7: track 0.00 -> 43.6 mm
- net Net-(D36-A): track 0.00 -> 5.60 mm
- net Net-(D35-A): track 0.00 -> 5.60 mm
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Other:
- board outline added: 168.9 x 134.6 mm
