File: kicad/Valmer 1.kicad_sch (KiCad schematic)
At the start: 75 parts, among them U1 RP2040_Pro_Micro

Commit message: kicad update
Connections:
- net Row 5 is gone; now on net Row 4: D30.1 (K), D31.1 (K), D32.1 (K), D33.1 (K), D34.1 (K), D35.1 (K), D36.1 (K), D37.1 (K)
- net Colum 0: now also U1.6 (GP2)
- net Colum 1: now also U1.7 (GP3)
- net Colum 2: now also U1.8 (GP4)
- net Colum 3: now also U1.9 (GP5)
- net Colum 4: now also U1.10 (GP6)
- net Colum 5: now also U1.11 (GP7)
- net Colum 6: now also U1.12 (GP8)
- net Colum 7: now also U1.13 (GP9)
- net Row 0: now also U1.31 (GP11)
- net Row 1: now also U1.1 (GP10)
- net Row 3: now also D22.1 (K), D23.1 (K), D24.1 (K), D25.1 (K), D26.1 (K), D27.1 (K), D28.1 (K), D29.1 (K), U1.15 (GP13); no longer D15.1 (K), D16.1 (K), D17.1 (K), D18.1 (K), D19.1 (K), D20.1 (K), D21.1 (K)
- net Row 4: now also U1.16 (GP14); no longer D22.1 (K), D23.1 (K), D24.1 (K), D25.1 (K), D26.1 (K), D27.1 (K), D28.1 (K), D29.1 (K)
- net Row 2: now reaches U1.14 (GP12)
- net Row 2: now also D15.1 (K), D16.1 (K), D17.1 (K), D18.1 (K), D19.1 (K), D20.1 (K), D21.1 (K)
- net GND: now reaches U1.29 (GND)
- net GND: now also U1.4 (GND), U1.5 (GND)
- net +5V: now reaches U1.30 (5v)
Other:
- added sheet LED Matrix (untitled.kicad_sch)
- moved on the sheet: U1
